File: HW/Spotify_controller.kicad_sch (KiCad schematic)
At the start: 52 parts, among them J1 Conn_02x04_Top_Bottom, J3 Conn_01x05_Socket, J4 USB_B_Micro, SW1 SW_Push, SW2 SW_Push, SW3 SW_Push, SW4 SW_Push, SW5 Boot, SW6 RotaryEncoder_Switch, U1 ESP32-C3-WROOM-02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

Commit message: add hw bugfixes
Parts:
- added A1, A2, A3, A4: M2.5 15mm, symbol Pia:Spacer/Abstandsbolzen
- added A10, A5, A6, A7, A8, A9: M2.5 10mm, symbol Pia:Spacer/Abstandsbolzen
- added D4, D5: 1N5819, Diode_THT:D_DO-41_SOD81_P7.62mm_Horizontal, symbol Diode:1N5819
- added J5: Conn_01x03, Connector_PinSocket_2.54mm:PinSocket_1x03_P2.54mm_Vertical, symbol Connector_Generic:Conn_01x03
- added J6, J7: Conn_01x09_Pin, Connector_PinHeader_1.27mm:PinHeader_1x09_P1.27mm_Vertical, symbol Connector:Conn_01x09_Pin
- added R15, R16: 300R, Resistor_THT:R_Axial_DIN0207_L6.3mm_D2.5mm_P10.16mm_Horizontal, symbol Device:R
- added S1, S10, S11, S12, S13, S14, S15, S16, S17, S18, S2, S3, S4, S5, S6, S7, S8, S9: M2.5, symbol Pia:Screw
- added SW7: SW_DIP_x01, Pia_Lib:Drahtschalter, symbol Switch:SW_DIP_x01
- 3V3: renamed from TP_3V3; value Bat+ -> 3V3; footprint Connector_Pin:Pin_D1.0mm_L10.0mm -> Connector_Pin:Pin_D1.3mm_L11.0mm
- C10: symbol Device:C -> Device:C_Polarized
- C11: footprint Capacitor_THT:C_Disc_D3.0mm_W2.0mm_P2.50mm -> Capacitor_THT:C_Disc_D4.7mm_W2.5mm_P5.00mm; now not fitted
- FID1, FID2, FID3, H1, H2, H3, H4, H5, H6: now left out of the parts list
- GND1: renamed from TP_GND1; value Bat+ -> GND; footprint Connector_Pin:Pin_D1.0mm_L10.0mm -> Connector_Pin:Pin_D1.3mm_L11.0mm
- J4, R8: now not fitted
- R11: value 22R -> 300R
- renumbered U3 to D6
Connections:
- net +3V3: now also J7.1 (Pin_1), SW7.2
- net Boot: now also J7.8 (Pin_8)
- net CLK/SCL: now also J7.5 (Pin_5)
- net ENC_CLK: now also J6.6 (Pin_6)
- net ENC_DT: now also J7.3 (Pin_3)
- net ENC_SW: now also J7.4 (Pin_4)
- net GND: now also C10.2, J5.3 (Pin_3), J7.9 (Pin_9); no longer C10.1
- net MOSI/SDA: now also J7.6 (Pin_6)
- net USB_DN: now also J6.4 (Pin_4)
- net USB_DP: now also J6.5 (Pin_5)
- net DUOLED_1: now reaches R2.1, U1.18 (GPIO0/ADC1_CH0/XTAL_32K_P)
- net DUOLED_1: now also J6.9 (Pin_9)
- net GPIO10: now reaches R6.1, U1.10 (GPIO10)
- net GPIO10: now also J6.1 (Pin_1)
- net GPIO2/LED: now reaches R1.1, U1.16 (GPIO2/ADC1_CH2)
- net GPIO2/LED: now also D4.1 (K), J6.7 (Pin_7)
- net DUOLED_2: now reaches R3.1, U1.17 (GPIO1/ADC1_CH1/XTAL_32K_N)
- net DUOLED_2: now also J6.8 (Pin_8)
- net EN: now reaches R5.2, R7.1, U1.2 (EN/CHIP_PU)
- net EN: now also C10.1, J7.2 (Pin_2); no longer C10.2
- net Button_Left: now reaches U1.7 (GPIO8)
- net Button_Left: now also R11.1, D5.1 (K), J7.7 (Pin_7); no longer R11.2
- net USR_BTN1 renamed RX/Button_Middle
- net RX/Button_Middle: now also J5.2 (Pin_2), J6.2 (Pin_2), R15.2; no longer SW1.1
- net USR_BTN2 renamed USR_BTN_LEFT
- net USR_BTN_LEFT: now also R11.2; no longer R11.1
- net USR_BTN3 renamed TX/Button_Right
- net TX/Button_Right: now also J5.1 (Pin_1), J6.3 (Pin_3), R16.2; no longer SW4.1
- new net Program1: D4.2 (A), D5.2 (A), SW7.1
- new net USR_BTN_MIDDLE: R15.1, SW1.1
- new net USR_BTN_RIGHT: R16.1, SW4.1
Other:
- note added: "Pia Piekarek"
- note added: "Spotify Controller V0.91"
- moved on the sheet: C12, C5, C6, D1, D6, FID1, FID2, FID3, H1, H2, H3, H4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

Commit message: add all current changes
Parts:
- added J2: Conn_01x04, Connector_PinSocket_2.54mm:PinSocket_1x04_P2.54mm_Vertical, symbol Connector_Generic:Conn_01x04
- D4, D5: footprint Diode_THT:D_DO-41_SOD81_P7.62mm_Horizontal -> Diode_THT:D_DO-41_SOD81_P10.16mm_Horizontal
- D6: value ~ -> Zweifarb-LED; footprint LED_THT:LED_D3.0mm-3 -> Pia_Lib:LED-3Pin
- R12, R13, R14: now not fitted
Connections:
- net +3V3: now also SW7.1, J2.2 (Pin_2); no longer SW7.2
- net CLK/SCL: now also J2.3 (Pin_3)
- net GND: now also J2.1 (Pin_1)
- net MOSI/SDA: now also J2.4 (Pin_4)
- net Program1: now also SW7.2; no longer SW7.1
Other:
- moved on the sheet: D6, SW7

Commit message: add minor changes to Schematic and PCB
Parts:
- added DSP1: ~, symbol Pia:Display_SSD1306_0,96
- J4: Order Link  (none) -> https://www.reichelt.de/usb-buchse-typ-micro-b-smd-gull-win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
Other:
- note added: "Alternative for programming"
- note added: "Either KY-040 Board or ALPS EC11"
- note added: "For Programming"
- note added: "If there are any Problems with the USB Connection while using the MicroUSB socket, please make a drill in the Dot that is marked in the PCB. These tracks will bring noise to the tracks otherwise."
- note added: "Using Internal Pullups and debouncing via SW"
Changed lines of the file:
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@@
     (stroke (width 0) (type default))
   )
-  (rectangle (start 15.24 200.025) (end 160.655 283.845)
+  (rectangle (start 15.24 200.025) (end 175.26 283.845)
     (stroke (width 0) (type default))
     (fill (type none))
   )
-  (rectangle (start 14.605 86.995) (end 194.31 199.39)
+  (rectangle (start 14.605 86.995) (end 180.34 199.39)
     (stroke (width 0) (type default))
     (fill (type none))
@@
     )
   )
-  (image (at 236.22 226.06) (scale 2.11268)
+  (image (at 240.665 233.045) (scale 2.11268)
     (data
       iVBORw0KGgoAAAANSUhEUgAAAokAAAJECAIAAAD1wykcAAAAA3NCSVQICAjb4U/gAAAACXBIWXMA
@@
     (effects (font (size 1.27 1.27)) (justify left bottom))
   )
+  (text "If there are any Problems with the USB Connection \nwhile using the MicroUSB socket, please make a drill \nin the Dot that is marked in the PCB. These tracks \nwill bring noise to the tracks otherwise."
+    (at 20.955 277.495 0)
+    (effects (font (size 1.27 1.27)) (justify left bottom))
+  )
   (text "alt 4k7" (at 163.195 153.67 0)
     (effects (font (size 1.27 1.27)) (justify left bottom))
   )
+  (text "Using Internal Pullups and debouncing via SW" (at 210.185 92.71 0)
+    (effects (font (size 1.27 1.27)) (justify left bottom))
+  )
+  (text "Alternative for programming" (at 137.795 92.075 0)
+    (effects (font (size 1.27 1.27)) (justify left bottom))
+  )
   (text "JTAG" (at 121.92 154.94 0)
     (effects (font (size 1.27 1.27)) (justify left bottom))
@@
     (effects (font (size 1.27 1.27)) (justify left bottom))
   )
+  (text "For Programming" (at 179.705 24.765 0)
+    (effects (font (size 1.27 1.27)) (justify left bottom))
+  )
   (text "USR BTN" (at 250.19 17.78 0)
     (effects (font (size 1.27 1.27)) (justify left bottom))
@@
     (effects (font (size 1.27 1.27)) (justify left bottom))
   )
+  (text "Either KY-040 Board or ALPS EC11" (at 245.11 137.16 0)
+    (effects (font (size 1.27 1.27)) (justify left bottom))
+  )
   (label "Boot" (at 150.495 160.655 0) (fields_autoplaced)
     (effects (font (size 1.27 1.27)) (justify left bottom))
@@
       (effects (font (size 1.27 1.27)) hide)
     )
+    (property "Order Link " "https://www.reichelt.de/usb-buchse-typ-micro-b-smd-gull-wing-mpe-712-1-s-bs0-p263308.html?PROVID=2788&gclid=CjwKCAiAvJarBhA1EiwAGgZl0NEqI-E8U4ifBROS_VqsahALfrSO3HXWrVPk3H4jfoQe-jLzNHP3yxoCJRgQAvD_BwE" (at 44.45 220.98 0)
+      (effects (font (size 1.27 1.27)) hide)
+    )
     (pin "1")
     (pin "2")
@@
         )
       )
+    )
+  )
+  (symbol (lib_id "Pia:Display_SSD1306_0,96") (at 142.875 215.265 0) (unit 1)
+    (in_bom yes) (on_board no) (dnp no)
+    (property "Reference" "DSP1" (at 140.97 222.885 0)
+      (effects (font (size 1.27 1.27)) (justify left))
+    )
+    (property "Value" "~" (at 142.875 215.265 0)
+      (effects (font (size 1.27 1.27)))
+    )
+    (property "Footprint" "" (at 142.875 215.265 0)
+      (effects (font (size 1.27 1.27)) hide)
+    )
+    (property "Datasheet" "https://www.az-delivery.de/products/0-96zolldisplay?variant=39457349828704" (at 142.875 215.265 0)
+      (effects (font (size 1.27 1.27)) hide)
+    )
+    (property "Alternative" "https://de.aliexpress.com/item/32809885818.html?src=google&src=google&albch=shopping&acnt=272-267-0231&slnk=&plac=&mtctp=&albbt=Google_7_shopping&gclsrc=aw.ds&albagn=888888&ds_e_adid=&ds_e_matchtype=&ds_e_device=c&ds_e_network=x&ds_e_product_group_id=&ds_e_product_id=de32809885818&ds_e_product_merchant_id=107694425&ds_e_product_country=DE&ds_e_product_language=de&ds_e_product_channel=online&ds_e_product_store_id=&ds_url_v=2&albcp=20701456946&albag=&isSmbAutoCall=false&needSmbHouyi=false&gad_source=1&gclid=CjwKCAiAvJarBhA1EiwAGgZl0HEzlgKkQtPhLsvHwdyh5cOqLLaGHSqxK8XKggfMNZ4WEQ4GYi3HrBoCI2IQAvD_BwE&aff_fcid=582898bbeedf41eb85a1d4355f4bc5ca-1701167417425-06431-UneMJZVf&aff_fsk=UneMJZVf&aff_platform=aaf&sk=UneMJZVf&aff_trace_key=582898bbeedf41eb85a1d4355f4bc5ca-1701167417425-06431-UneMJZVf&terminal_id=bd387386fe044ce39da61f5fa04ea958&afSmartRedirect=y" (at 142.875 215.265 0)
+      (effects (font (size 1.27 1.27)) hide)
+    )
+    (instances
+      (project "Spotify_controller"
+        (path "/5b72fb14-a995-4a92-8291-dd28bff636b0"
+          (reference "DSP1") (unit 1)
+        )
+      )
