File: HW/Spotify_controller.kicad_sch (KiCad schematic)
At the start: 90 parts, among them J1 Conn_02x04_Top_Bottom, J2 Conn_01x04, J3 Conn_01x05_Socket, J4 USB_B_Micro, J5 Conn_01x03, J6 Conn_01x09_Pin, J7 Conn_01x09_Pin, SW1 SW_Push, SW2 SW_Push, SW3 SW_Push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

Commit message: add minor changes
Parts:
- renumbered 3V3 to 3V3?
Changed lines of the file:
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@@
   (symbol (lib_id "Connector:TestPoint") (at 85.725 33.02 0) (unit 1)
     (in_bom yes) (on_board yes) (dnp no) (fields_autoplaced)
-    (property "Reference" "3V3" (at 87.63 29.083 0)
+    (property "Reference" "3V3?" (at 87.63 29.083 0)
       (effects (font (size 1.27 1.27)) (justify left))
     )
@@
       (project "Spotify_controller"
         (path "/5b72fb14-a995-4a92-8291-dd28bff636b0"
-          (reference "3V3") (unit 1)
+          (reference "3V3?") (unit 1)
         )
       )

Commit message: additional minor changes
Parts:
- gave numbers to parts that had none: 1
Changed lines of the file:
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@@
   (symbol (lib_id "Connector:TestPoint") (at 85.725 33.02 0) (unit 1)
     (in_bom yes) (on_board yes) (dnp no) (fields_autoplaced)
-    (property "Reference" "3V3?" (at 87.63 29.083 0)
+    (property "Reference" "3V31" (at 87.63 29.083 0)
       (effects (font (size 1.27 1.27)) (justify left))
     )
@@
       (project "Spotify_controller"
         (path "/5b72fb14-a995-4a92-8291-dd28bff636b0"
-          (reference "3V3?") (unit 1)
+          (reference "3V31") (unit 1)
         )
       )

Commit message: minor changes 2
Parts:
- renumbered GND1 to TP3, 3V31 to TP4
Changed lines of the file:
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@@
   (symbol (lib_id "Connector:TestPoint") (at 85.725 33.02 0) (unit 1)
     (in_bom yes) (on_board yes) (dnp no) (fields_autoplaced)
-    (property "Reference" "3V31" (at 87.63 29.083 0)
+    (property "Reference" "TP4" (at 87.63 29.083 0)
       (effects (font (size 1.27 1.27)) (justify left))
     )
@@
       (project "Spotify_controller"
         (path "/5b72fb14-a995-4a92-8291-dd28bff636b0"
-          (reference "3V31") (unit 1)
+          (reference "TP4") (unit 1)
         )
       )
@@
   (symbol (lib_id "Connector:TestPoint") (at 85.09 48.26 180) (unit 1)
     (in_bom yes) (on_board yes) (dnp no) (fields_autoplaced)
-    (property "Reference" "GND1" (at 87.63 50.927 0)
+    (property "Reference" "TP3" (at 87.63 50.927 0)
       (effects (font (size 1.27 1.27)) (justify right))
     )
@@
       (project "Spotify_controller"
         (path "/5b72fb14-a995-4a92-8291-dd28bff636b0"
-          (reference "GND1") (unit 1)
-        )
-      )
+          (reference "TP3") (unit 1)
+        )
+      )
