File: HW/Spotify_controller.kicad_pcb (KiCad board)
At the start: 2 copper layers, 38 x 100 mm, 52 parts, among them J1 Conn_02x04_Top_Bottom, J3 Conn_01x05_Socket, J4 USB_B_Micro, SW1 SW_Push, SW2 SW_Push, SW3 SW_Push, SW4 SW_Push, SW5 Boot, SW6 RotaryEncoder_Switch, U1 ESP32-C3-WROOM-02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

Commit message: add hw bugfixes
Parts:
- removed TP_3V3, TP_GND1: Bat+, Connector_Pin:Pin_D1.0mm_L10.0mm
- removed U3: ~, LED_THT:LED_D3.0mm-3
- added 3V3: 3V3, Connector_Pin:Pin_D1.3mm_L11.0mm, F.Cu at (57.4, 50.6)
- added D4: 1N5819, Diode_THT:D_DO-41_SOD81_P7.62mm_Horizontal, F.Cu at (30.7, 127.3)
- added D5: 1N5819, Diode_THT:D_DO-41_SOD81_P7.62mm_Horizontal, F.Cu at (44.0, 113.0)
- added D6: ~, LED_THT:LED_D3.0mm-3, F.Cu at (40.0, 77.7)
- added G***: LOGO, LOGO, B.Cu at (44.9, 102.1)
- added G***: LOGO, LOGO, B.Cu at (62.4, 48.9)
- added G***: LOGO, Pia_Lib:QRCode1x1, B.Cu at (45.4, 128.8)
- added GND1: GND, Connector_Pin:Pin_D1.3mm_L11.0mm, F.Cu at (57.3, 44.5)
- added J5: Conn_01x03, Connector_PinSocket_2.54mm:PinSocket_1x03_P2.54mm_Vertical, F.Cu at (30.1, 110.4)
- added J6: Conn_01x09_Pin, Connector_PinHeader_1.27mm:PinHeader_1x09_P1.27mm_Vertical, F.Cu at (35.1, 123.7)
- added J7: Conn_01x09_Pin, Connector_PinHeader_1.27mm:PinHeader_1x09_P1.27mm_Vertical, F.Cu at (59.2, 133.9)
- added R15: 300R, Resistor_THT:R_Axial_DIN0207_L6.3mm_D2.5mm_P10.16mm_Horizontal, F.Cu at (33.6, 97.2)
- added R16: 300R, Resistor_THT:R_Axial_DIN0207_L6.3mm_D2.5mm_P10.16mm_Horizontal, F.Cu at (30.6, 97.2)
- added SW7: SW_DIP_x01, Pia_Lib:Drahtschalter, F.Cu at (41.2, 115.0)
- C11: footprint Capacitor_THT:C_Disc_D3.0mm_W2.0mm_P2.50mm -> Capacitor_THT:C_Disc_D4.7mm_W2.5mm_P5.00mm
- R11: value 22R -> 300R
- moved FID1 6.55 mm to (36.9, 44.2)
- moved R12 3.24 mm to (52.9, 132.6)
- moved R14 3.23 mm to (52.9, 130.6)
- moved R4 1.78 mm to (58.0, 107.3)
- moved R2 1.78 mm to (51.9, 107.3)
- moved R1 1.77 mm to (55.0, 107.3)
- moved R3 1.75 mm to (48.9, 107.3)
- moved R6 1.73 mm to (45.8, 107.3)
- moved R11 1.71 mm to (42.8, 97.2)
- moved R10 1.69 mm to (39.7, 97.2)
- moved R9 1.68 mm to (36.7, 97.2)
- moved C10 1.02 mm to (62.6, 124.0)
- moved C11 0.13 mm to (33.1, 44.0)
- moved SW3 0.09 mm to (35.9, 88.0)
Connections:
- net Net-(U1-GPIO0/ADC1_CH0/XTAL_32K_P) renamed /DUOLED_1
- net Net-(U1-GPIO10) renamed /GPIO10
- net Net-(U1-GPIO1/ADC1_CH1/XTAL_32K_N) renamed /DUOLED_2
- net Net-(U1-GPIO2/ADC1_CH2) renamed /GPIO2/LED
- net Net-(U1-GPIO8) renamed /Button_Left
- net USR_BTN2 renamed USR_BTN_LEFT
- C10 pad 1: GND -> /EN
- C10 pad 2: Net-(U1-EN/CHIP_PU) -> GND
- R5 pad 2: Net-(U1-EN/CHIP_PU) -> /EN
- R7 pad 1: Net-(U1-EN/CHIP_PU) -> /EN
- SW1 pad 1: USR_BTN1 -> USR_BTN_MIDDLE
- SW4 pad 1: USR_BTN3 -> USR_BTN_RIGHT
- U1 pad 11: USR_BTN1 -> /RX/Button_Middle
- U1 pad 12: USR_BTN3 -> /TX/Button_Right
- U1 pad 2: Net-(U1-EN/CHIP_PU) -> /EN
Routing:
- net USR_BTN3: track 81.7 -> 0.00 mm, vias 3 -> 0
- net USR_BTN1: track 67.9 -> 0.00 mm, vias 1 -> 0
- net USR_BTN_RIGHT: track 0.00 -> 64.3 mm, vias 0 -> 3
- net USR_BTN_MIDDLE: track 0.00 -> 44.0 mm, vias 0 -> 1
- net /Program1: track 0.00 -> 38.0 mm, vias 0 -> 2
- net Net-(U1-EN/CHIP_PU): track 28.5 -> 0.00 mm
- net /EN: track 0.00 -> 28.0 mm
- net /TX/Button_Right: track 0.00 -> 26.9 mm, vias 0 -> 1
- net /RX/Button_Middle: track 0.00 -> 25.6 mm, vias 0 -> 1
- net /D+: track 110.9 -> 86.4 mm, vias 1 -> 3
- net GND: track 373.9 -> 396.3 mm
- net /GPIO2/LED: track 36.2 -> 48.2 mm
- net CLK/SCL: track 94.6 -> 104.0 mm
- net USB_DP: track 37.0 -> 28.6 mm
- net VBUS: track 43.1 -> 51.0 mm
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Other:
- board text added: "+"
- board text added: "Boot"
- board text added: "EN"
- board text added: "G"
- board text added: "Prog"
- board text added: "RX"
- board text added: "TX"
- board text added: "https://github.com/RT-CUSTOMZ/ Spotify-Controller/wiki"

Commit message: add all current changes
Parts:
- added J2: Conn_01x04, Connector_PinSocket_2.54mm:PinSocket_1x04_P2.54mm_Vertical, F.Cu at (64.2, 44.8)
- D4, D5: footprint Diode_THT:D_DO-41_SOD81_P7.62mm_Horizontal -> Diode_THT:D_DO-41_SOD81_P10.16mm_Horizontal
- D6: value ~ -> Zweifarb-LED; footprint LED_THT:LED_D3.0mm-3 -> Pia_Lib:LED-3Pin
- G***: moved to F.Cu
- moved G*** 55.0 mm to (62.8, 103.9), turned to 0 degrees
- moved R11 10.2 mm to (42.8, 107.3), turned to 90 degrees
- moved SW7 5.99 mm to (35.3, 116.0), turned to 90 degrees
- moved FID1 4.44 mm to (41.1, 45.6)
- moved D6 2.58 mm to (42.6, 77.6)
- moved D5 2.57 mm to (44.0, 110.4)
- moved D4 2.24 mm to (30.6, 125.0)
Connections:
- R11 pad 1: USR_BTN_LEFT -> /Button_Left
- R11 pad 2: /Button_Left -> /USR_BTN_LEFT
- SW3 pad 1: USR_BTN_LEFT -> /USR_BTN_LEFT
- SW7 pad 1: /Program1 -> +3V3
- SW7 pad 2: +3V3 -> /Program1
Routing:
- net CLK/SCL: track 104.0 -> 133.3 mm
- net MOSI/SDA: track 111.0 -> 139.0 mm, vias 3 -> 5
- net USR_BTN_LEFT: track 19.4 -> 0.00 mm
- net /USR_BTN_LEFT: track 0.00 -> 18.8 mm
- net USR_BTN_RIGHT: track 64.3 -> 56.3 mm
- net VBUS: track 51.0 -> 43.6 mm
- net +3V3: track 160.0 -> 166.9 mm
- net GND: track 396.3 -> 402.0 mm
- net /D+: track 86.4 -> 81.8 mm
- net /D-: track 68.6 -> 64.3 mm
- net /DUOLED_2: track 38.8 -> 35.1 mm, vias 1 -> 0
- net /DUOLED_1: track 42.6 -> 38.8 mm, vias 1 -> 0
- net /Button_Left: track 36.6 -> 33.1 mm, vias 2 -> 1
- net ENC_CLK: track 105.6 -> 102.5 mm
- net /GPIO2/LED: track 48.2 -> 51.2 mm
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Other:
- board text added: "V1.0"
- board text removed: "V0.91"

Commit message: Manufacturing Data for JLCPCB generated
Parts:
- moved GND1 0.23 mm to (57.2, 44.7)
Routing:
- net ENC_DT: track 112.6 -> 112.1 mm
Other:
- board text added: "Remotify V1.0"
- board text removed: "Spotify Controller"
- board text removed: "V1.0"

Commit message: add minor changes
Parts:
- added 3V31: 3V3, Connector_Pin:Pin_D1.3mm_L11.0mm, F.Cu at (57.4, 50.6)
Changed lines of the file:
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@@
+  )
+  (footprint "Connector_Pin:Pin_D1.3mm_L11.0mm" (layer "F.Cu")
+    (at 57.4294 50.6476)
+    (descr "solder Pin_ diameter 1.3mm, hole diameter 1.3mm, length 11.0mm")
+    (tags "solder Pin_ pressfit")
+    (property "Sheetfile" "Spotify_controller.kicad_sch")
+    (property "Sheetname" "")
+    (property "ki_description" "test point")
+    (property "ki_keywords" "test point tp")
+    (attr through_hole)
+    (fp_text reference "3V31" (at 0 2.4) (layer "F.SilkS")
+        (effects (font (size 1 1) (thickness 0.15)))
+    )
+    (fp_text value "3V3" (at 0 -2.05) (layer "F.Fab")
+        (effects (font (size 1 1) (thickness 0.15)))
+    )
+    (fp_text user "${REFERENCE}" (at 0 2.4) (layer "F.Fab")
+        (effects (font (size 1 1) (thickness 0.15)))
+    )
+    (fp_circle (center 0 0) (end 1.6 0.05)
+      (stroke (width 0.12) (type solid)) (fill none) (layer "F.SilkS"))
+    (fp_circle (center 0 0) (end 1.8 0)
+      (stroke (width 0.05) (type solid)) (fill none) (layer "F.CrtYd"))
+    (fp_circle (center 0 0) (end 0.65 -0.05)
+      (stroke (width 0.12) (type solid)) (fill none) (layer "F.Fab"))
+    (fp_circle (center 0 0) (end 1.25 -0.05)
+      (stroke (width 0.12) (type solid)) (fill none) (layer "F.Fab"))
+    (pad "1" thru_hole circle (at 0 0) (size 2.6 2.6) (drill 1.3) (layers "*.Cu" "*.Mask")
+      (net 3 "+3V3") (pinfunction "1") (pintype "passive"))
+    (model "${KICAD6_3DMODEL_DIR}/Connector_Pin.3dshapes/Pin_D1.3mm_L11.0mm.wrl"
+      (offset (xyz 0 0 0))
+      (scale (xyz 1 1 1))
+      (rotate (xyz 0 0 0))
+    )
   )
   (footprint "Connector_Pin:Pin_D1.3mm_L11.0mm" (layer "F.Cu")

Commit message: additional minor changes
Parts:
- removed 3V3: 3V3, Connector_Pin:Pin_D1.3mm_L11.0mm
Changed lines of the file:
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@@
-    )
-  )
-  (footprint "Connector_Pin:Pin_D1.3mm_L11.0mm" (layer "F.Cu")
-    (at 57.4294 50.6476 180)
-    (descr "solder Pin_ diameter 1.3mm, hole diameter 1.3mm, length 11.0mm")
-    (tags "solder Pin_ pressfit")
-    (property "Sheetfile" "Spotify_controller.kicad_sch")
-    (property "Sheetname" "")
-    (property "ki_description" "test point")
-    (property "ki_keywords" "test point tp")
-    (attr through_hole)
-    (fp_text reference "3V3" (at 2.8702 1.3208) (layer "F.SilkS")
-        (effects (font (size 1 1) (thickness 0.15)))
-    )
-    (fp_text value "3V3" (at 0 -2.05) (layer "F.Fab")
-        (effects (font (size 1 1) (thickness 0.15)))
-    )
-    (fp_text user "${REFERENCE}" (at 0 2.4) (layer "F.Fab")
-        (effects (font (size 1 1) (thickness 0.15)))
-    )
-    (fp_circle (center 0 0) (end 1.6 0.05)
-      (stroke (width 0.12) (type solid)) (fill none) (layer "F.SilkS"))
-    (fp_circle (center 0 0) (end 1.8 0)
-      (stroke (width 0.05) (type solid)) (fill none) (layer "F.CrtYd"))
-    (fp_circle (center 0 0) (end 0.65 -0.05)
-      (stroke (width 0.12) (type solid)) (fill none) (layer "F.Fab"))
-    (fp_circle (center 0 0) (end 1.25 -0.05)
-      (stroke (width 0.12) (type solid)) (fill none) (layer "F.Fab"))
-    (pad "1" thru_hole circle (at 0 0 180) (size 2.6 2.6) (drill 1.3) (layers "*.Cu" "*.Mask")
-      (net 3 "+3V3") (pinfunction "1") (pintype "passive"))
-    (model "${KICAD6_3DMODEL_DIR}/Connector_Pin.3dshapes/Pin_D1.3mm_L11.0mm.wrl"
-      (offset (xyz 0 0 0))
-      (scale (xyz 1 1 1))
-      (rotate (xyz 0 0 0))
     )
   )

Commit message: minor changes 2
Parts:
- removed 3V31: 3V3, Connector_Pin:Pin_D1.3mm_L11.0mm
- removed GND1: GND, Connector_Pin:Pin_D1.3mm_L11.0mm
- added TP3: GND, Connector_Pin:Pin_D1.3mm_L11.0mm, F.Cu at (57.1, 44.7)
- added TP4: 3V3, Connector_Pin:Pin_D1.3mm_L11.0mm, F.Cu at (57.4, 50.6)
Changed lines of the file:
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@@
     )
   )
+  (footprint "Connector_Pin:Pin_D1.3mm_L11.0mm" (layer "F.Cu")
+    (at 57.1246 44.704)
+    (descr "solder Pin_ diameter 1.3mm, hole diameter 1.3mm, length 11.0mm")
+    (tags "solder Pin_ pressfit")
+    (property "Sheetfile" "Spotify_controller.kicad_sch")
+    (property "Sheetname" "")
+    (property "ki_description" "test point")
+    (property "ki_keywords" "test point tp")
+    (attr through_hole)
+    (fp_text reference "TP3" (at 3.2512 0.2794) (layer "F.SilkS") hide
+        (effects (font (size 1 1) (thickness 0.15)))
+    )
+    (fp_text value "GND" (at 0 -2.05) (layer "F.Fab")
+        (effects (font (size 1 1) (thickness 0.15)))
+    )
+    (fp_text user "${REFERENCE}" (at 0 2.4) (layer "F.Fab")
+        (effects (font (size 1 1) (thickness 0.15)))
+    )
+    (fp_circle (center 0 0) (end 1.6 0.05)
+      (stroke (width 0.12) (type solid)) (fill none) (layer "F.SilkS"))
+    (fp_circle (center 0 0) (end 1.8 0)
+      (stroke (width 0.05) (type solid)) (fill none) (layer "F.CrtYd"))
+    (fp_circle (center 0 0) (end 0.65 -0.05)
+      (stroke (width 0.12) (type solid)) (fill none) (layer "F.Fab"))
+    (fp_circle (center 0 0) (end 1.25 -0.05)
+      (stroke (width 0.12) (type solid)) (fill none) (layer "F.Fab"))
+    (pad "1" thru_hole circle (at 0 0) (size 2.6 2.6) (drill 1.3) (layers "*.Cu" "*.Mask")
+      (net 2 "GND") (pinfunction "1") (pintype "passive"))
+    (model "${KICAD6_3DMODEL_DIR}/Connector_Pin.3dshapes/Pin_D1.3mm_L11.0mm.wrl"
+      (offset (xyz 0 0 0))
+      (scale (xyz 1 1 1))
+      (rotate (xyz 0 0 0))
+    )
+  )
   (footprint "Resistor_THT:R_Axial_DIN0207_L6.3mm_D2.5mm_P10.16mm_Horizontal" (layer "F.Cu")
     (at 51.9176 107.3404 90)
@@
     )
   )
-  (footprint "Connector_Pin:Pin_D1.3mm_L11.0mm" (layer "F.Cu")
-    (at 57.4294 50.6476)
-    (descr "solder Pin_ diameter 1.3mm, hole diameter 1.3mm, length 11.0mm")
-    (tags "solder Pin_ pressfit")
-    (property "Sheetfile" "Spotify_controller.kicad_sch")
-    (property "Sheetname" "")
-    (property "ki_description" "test point")
-    (property "ki_keywords" "test point tp")
-    (attr through_hole)
-    (fp_text reference "3V31" (at 0 2.4) (layer "F.SilkS")
-        (effects (font (size 1 1) (thickness 0.15)))
-    )
-    (fp_text value "3V3" (at 0 -2.05) (layer "F.Fab")
-        (effects (font (size 1 1) (thickness 0.15)))
-    )
-    (fp_text user "${REFERENCE}" (at 0 2.4) (layer "F.Fab")
-        (effects (font (size 1 1) (thickness 0.15)))
-    )
-    (fp_circle (center 0 0) (end 1.6 0.05)
-      (stroke (width 0.12) (type solid)) (fill none) (layer "F.SilkS"))
-    (fp_circle (center 0 0) (end 1.8 0)
-      (stroke (width 0.05) (type solid)) (fill none) (layer "F.CrtYd"))
-    (fp_circle (center 0 0) (end 0.65 -0.05)
-      (stroke (width 0.12) (type solid)) (fill none) (layer "F.Fab"))
-    (fp_circle (center 0 0) (end 1.25 -0.05)
-      (stroke (width 0.12) (type solid)) (fill none) (layer "F.Fab"))
-    (pad "1" thru_hole circle (at 0 0) (size 2.6 2.6) (drill 1.3) (layers "*.Cu" "*.Mask")
-      (net 3 "+3V3") (pinfunction "1") (pintype "passive"))
-    (model "${KICAD6_3DMODEL_DIR}/Connector_Pin.3dshapes/Pin_D1.3mm_L11.0mm.wrl"
-      (offset (xyz 0 0 0))
-      (scale (xyz 1 1 1))
-      (rotate (xyz 0 0 0))
-    )
-  )
   (footprint "Pia_Lib:Drahtschalter" (layer "F.Cu")
     (at 35.306 116.0272 90)
@@
     )
   )
-  (footprint "Connector_Pin:Pin_D1.3mm_L11.0mm" (layer "F.Cu")
-    (at 57.2262 44.704)
-    (descr "solder Pin_ diameter 1.3mm, hole diameter 1.3mm, length 11.0mm")
-    (tags "solder Pin_ pressfit")
-    (property "Sheetfile" "Spotify_controller.kicad_sch")
-    (property "Sheetname" "")
-    (property "ki_description" "test point")
-    (property "ki_keywords" "test point tp")
-    (attr through_hole)
-    (fp_text reference "GND1" (at -3.5306 -1.2446) (layer "F.SilkS")
-        (effects (font (size 1 1) (thickness 0.15)))
-    )
-    (fp_text value "GND" (at 0 -2.05) (layer "F.Fab")
-        (effects (font (size 1 1) (thickness 0.15)))
-    )
-    (fp_text user "${REFERENCE}" (at 0 2.4) (layer "F.Fab")
-        (effects (font (size 1 1) (thickness 0.15)))
-    )
-    (fp_circle (center 0 0) (end 1.6 0.05)
-      (stroke (width 0.12) (type solid)) (fill none) (layer "F.SilkS"))
-    (fp_circle (center 0 0) (end 1.8 0)
-      (stroke (width 0.05) (type solid)) (fill none) (layer "F.CrtYd"))
-    (fp_circle (center 0 0) (end 0.65 -0.05)
-      (stroke (width 0.12) (type solid)) (fill none) (layer "F.Fab"))
-    (fp_circle (center 0 0) (end 1.25 -0.05)
-      (stroke (width 0.12) (type solid)) (fill none) (layer "F.Fab"))
-    (pad "1" thru_hole circle (at 0 0) (size 2.6 2.6) (drill 1.3) (layers "*.Cu" "*.Mask")
-      (net 2 "GND") (pinfunction "1") (pintype "passive"))
-    (model "${KICAD6_3DMODEL_DIR}/Connector_Pin.3dshapes/Pin_D1.3mm_L11.0mm.wrl"
-      (offset (xyz 0 0 0))
-      (scale (xyz 1 1 1))
-      (rotate (xyz 0 0 0))
-    )
-  )
   (footprint "Resistor_THT:R_Axial_DIN0207_L6.3mm_D2.5mm_P10.16mm_Horizontal" (layer "F.Cu")
     (at 45.8216 107.3404 90)
@@
     )
   )
+  (footprint "Connector_Pin:Pin_D1.3mm_L11.0mm" (layer "F.Cu")
+    (at 57.4294 50.6476)
+    (descr "solder Pin_ diameter 1.3mm, hole diameter 1.3mm, length 11.0mm")
+    (tags "solder Pin_ pressfit")
+    (property "Sheetfile" "Spotify_controller.kicad_sch")
+    (property "Sheetname" "")
+    (property "ki_description" "test point")
+    (property "ki_keywords" "test point tp")
+    (attr through_hole)
+    (fp_text reference "TP4" (at 3.1242 0.3048) (layer "F.SilkS") hide
+        (effects (font (size 1 1) (thickness 0.15)))
+    )
+    (fp_text value "3V3" (at 0 -2.05) (layer "F.Fab")
+        (effects (font (size 1 1) (thickness 0.15)))
+    )
+    (fp_text user "${REFERENCE}" (at 0 2.4) (layer "F.Fab")
+        (effects (font (size 1 1) (thickness 0.15)))
+    )
+    (fp_circle (center 0 0) (end 1.6 0.05)
+      (stroke (width 0.12) (type solid)) (fill none) (layer "F.SilkS"))
+    (fp_circle (center 0 0) (end 1.8 0)
+      (stroke (width 0.05) (type solid)) (fill none) (layer "F.CrtYd"))
+    (fp_circle (center 0 0) (end 0.65 -0.05)
+      (stroke (width 0.12) (type solid)) (fill none) (layer "F.Fab"))
+    (fp_circle (center 0 0) (end 1.25 -0.05)
+      (stroke (width 0.12) (type solid)) (fill none) (layer "F.Fab"))
+    (pad "1" thru_hole circle (at 0 0) (size 2.6 2.6) (drill 1.3) (layers "*.Cu" "*.Mask")
+      (net 3 "+3V3") (pinfunction "1") (pintype "passive"))
+    (model "${KICAD6_3DMODEL_DIR}/Connector_Pin.3dshapes/Pin_D1.3mm_L11.0mm.wrl"
+      (offset (xyz 0 0 0))
+      (scale (xyz 1 1 1))
+      (rotate (xyz 0 0 0))
+    )
+  )
   (footprint "MountingHole:MountingHole_2.7mm_M2.5" (layer "B.Cu")
     (at 63.45 74.36 180)
@@
   (segment (start 30.07 43.859999) (end 32.980799 43.859999) (width 0.4) (layer "F.Cu") (net 2))
   (segment (start 50.927 48.4378) (end 49.3944 46.9052) (width 0.4) (layer "F.Cu") (net 2))
+  (segment (start 57.1246 44.704) (end 57.2262 44.704) (width 0.4) (layer "F.Cu") (net 2))
   (segment (start 42.333598 46.9424) (end 37.4396 51.836398) (width 0.4) (layer "F.Cu") (net 2))
   (segment (start 47.245601 92.858999) (end 48.905002 92.858999) (width 0.4) (layer "F.Cu") (net 2))
